File: v2.1/zdrojV21.brd (EAGLE design)
At the start: 160 x 100 mm, 26 parts, among them IC1 LM358N, IC2 LM317, Q1 BS170

Commit message: pokračování v základním návrhu
Connections:
- removed net N$4: IC2.1, R4.2
- new net N$5: C3.+, D2.A, IC2.1, R4.2, R4.3, R5.1
- net GND: no longer C3.+, D2.A, R4.3, R5.1
Changed lines of the file:
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@@
 <contactref element="R7" pad="2"/>
 <contactref element="R4" pad="1"/>
-<contactref element="R4" pad="3"/>
-<contactref element="R5" pad="1"/>
-<contactref element="D2" pad="A"/>
 <contactref element="C2" pad="-"/>
 <contactref element="C3" pad="-"/>
-<contactref element="C3" pad="+"/>
 <contactref element="C1" pad="-"/>
 <contactref element="U$2" pad="2"/>
@@
 <wire x1="-26.67" y1="20.32" x2="-25.4" y2="17.78" width="0" layer="19" extent="1-1"/>
 <wire x1="-21.59" y1="22.86" x2="-26.67" y2="20.32" width="0" layer="19" extent="1-1"/>
-<wire x1="-19.05" y1="25.4" x2="-21.59" y2="22.86" width="0" layer="19" extent="1-1"/>
-<wire x1="-26.67" y1="34.29" x2="-19.05" y2="25.4" width="0" layer="19" extent="1-1"/>
-<wire x1="-26.67" y1="40.64" x2="-26.67" y2="34.29" width="0" layer="19" extent="1-1"/>
-<wire x1="-29.21" y1="40.64" x2="-26.67" y2="40.64" width="0" layer="19" extent="1-1"/>
-<wire x1="-24.13" y1="46.99" x2="-26.67" y2="40.64" width="0" layer="19" extent="1-1"/>
-<wire x1="-17.78" y1="40.64" x2="-26.67" y2="40.64" width="0" layer="19" extent="1-1"/>
-<wire x1="-43.18" y1="33.02" x2="-29.21" y2="40.64" width="0" layer="19" extent="1-1"/>
+<wire x1="-17.78" y1="40.64" x2="-21.59" y2="22.86" width="0" layer="19" extent="1-1"/>
+<wire x1="-26.67" y1="40.64" x2="-17.78" y2="40.64" width="0" layer="19" extent="1-1"/>
+<wire x1="-43.18" y1="33.02" x2="-26.67" y2="40.64" width="0" layer="19" extent="1-1"/>
 <wire x1="-49.53" y1="40.64" x2="-43.18" y2="33.02" width="0" layer="19" extent="1-1"/>
 <wire x1="-44.45" y1="46.99" x2="-49.53" y2="40.64" width="0" layer="19" extent="1-1"/>
@@
 <wire x1="-45.72" y1="2.54" x2="-62.23" y2="-8.89" width="0" layer="19" extent="1-1"/>
 </signal>
-<signal name="N$4">
-<contactref element="R4" pad="2"/>
-<contactref element="IC2" pad="1"/>
-<wire x1="-16.51" y1="22.86" x2="-45.72" y2="24.13" width="0" layer="19" extent="1-1"/>
-</signal>
 <signal name="V+-REG">
 <contactref element="R5" pad="2"/>
@@
 <wire x1="-38.1" y1="17.78" x2="-66.04" y2="-57.785" width="0" layer="19" extent="1-1"/>
 </signal>
+<signal name="N$5">
+<contactref element="R4" pad="3"/>
+<contactref element="R5" pad="1"/>
+<contactref element="D2" pad="A"/>
+<contactref element="C3" pad="+"/>
+<contactref element="R4" pad="2"/>
+<contactref element="IC2" pad="1"/>
+<wire x1="-29.21" y1="40.64" x2="-24.13" y2="46.99" width="0" layer="19" extent="1-1"/>
+<wire x1="-26.67" y1="34.29" x2="-29.21" y2="40.64" width="0" layer="19" extent="1-1"/>
+<wire x1="-19.05" y1="25.4" x2="-26.67" y2="34.29" width="0" layer="19" extent="1-1"/>
+<wire x1="-16.51" y1="22.86" x2="-19.05" y2="25.4" width="0" layer="19" extent="1-1"/>
+<wire x1="-45.72" y1="24.13" x2="-26.67" y2="34.29" width="0" layer="19" extent="1-1"/>
+</signal>
 </signals>
