File: v3.0/ovládací panel.brd (EAGLE design)
At the start: 100.3 x 32.7 mm, 6 parts

Commit message: Voila a enkodér funguje
Parts:
- added C1, C2: (no value), rcl:C0805
Connections:
- net GND: now also C1.2, C2.2
- net N$5: now also C2.1
- net N$6: now also C1.1
Changed lines of the file:
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@@
 <attribute name="VALUE" x="11.43" y="84.455" size="1.27" layer="27"/>
+</element>
+<element name="C1" library="rcl" library_urn="urn:adsk.eagle:library:334" package="C0805" package3d_urn="urn:adsk.eagle:package:23617/2" value="" x="-10.16" y="8.89" smashed="yes">
+<attribute name="NAME" x="-11.43" y="10.16" size="1.27" layer="25"/>
+<attribute name="POPULARITY" value="88" x="-10.16" y="8.89" size="1.778" layer="27" display="off"/>
+<attribute name="SPICEPREFIX" value="C" x="-10.16" y="8.89" size="1.778" layer="27" display="off"/>
+<attribute name="VALUE" x="-11.43" y="6.35" size="1.27" layer="27"/>
+</element>
+<element name="C2" library="rcl" library_urn="urn:adsk.eagle:library:334" package="C0805" package3d_urn="urn:adsk.eagle:package:23617/2" value="" x="-10.16" y="3.81" smashed="yes">
+<attribute name="NAME" x="-11.43" y="5.08" size="1.27" layer="25"/>
+<attribute name="POPULARITY" value="88" x="-10.16" y="3.81" size="1.778" layer="27" display="off"/>
+<attribute name="SPICEPREFIX" value="C" x="-10.16" y="3.81" size="1.778" layer="27" display="off"/>
+<attribute name="VALUE" x="-11.43" y="1.27" size="1.27" layer="27"/>
 </element>
 </elements>
@@
 <wire x1="57.15" y1="81.28" x2="59.56" y2="83.69" width="0.1524" layer="16"/>
 <wire x1="49.53" y1="85.09" x2="53.34" y2="81.28" width="0.1524" layer="1"/>
+<contactref element="C1" pad="2"/>
+<contactref element="C2" pad="2"/>
+<wire x1="-9.21" y1="8.89" x2="60.2488" y2="77.1906" width="0" layer="19" extent="1-1"/>
+<wire x1="-9.21" y1="3.81" x2="-9.21" y2="8.89" width="0" layer="19" extent="1-1"/>
 </signal>
 <signal name="GND1">
@@
 <wire x1="59.35" y1="93.9" x2="55.46" y2="97.79" width="0.8128" layer="16"/>
 <wire x1="55.46" y1="97.79" x2="54.61" y2="97.79" width="0.8128" layer="16"/>
+<contactref element="C2" pad="1"/>
+<wire x1="-11.11" y1="3.81" x2="34.29" y2="92.71" width="0" layer="19" extent="1-1"/>
 </signal>
 <signal name="N$6">
@@
 <wire x1="52.07" y1="96.52" x2="40.64" y2="96.52" width="0.8128" layer="1"/>
 <wire x1="40.64" y1="96.52" x2="36.83" y2="92.71" width="0.8128" layer="1"/>
+<contactref element="C1" pad="1"/>
+<wire x1="-11.11" y1="8.89" x2="36.83" y2="92.71" width="0" layer="19" extent="1-1"/>
 </signal>
 <signal name="N$7">
