File: v3.0/ovládací panel.sch (EAGLE design)
At the start: 6 parts

Commit message: Voila a enkodér funguje
Parts:
- added C1, C2: (no value), rcl:C-EUC0805
Connections:
- net GND: now also C1.2, C2.2
- net N$5: now also C2.1
- net N$6: now also C1.1
Changed lines of the file:
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@@
 <part name="GND6" library="supply1" library_urn="urn:adsk.eagle:library:371" deviceset="GND" device=""/>
 <part name="JP1" library="pinhead" library_urn="urn:adsk.eagle:library:325" deviceset="PINHD-1X4" device="" package3d_urn="urn:adsk.eagle:package:22407/2"/>
+<part name="C1" library="rcl" library_urn="urn:adsk.eagle:library:334" deviceset="C-EU" device="C0805" package3d_urn="urn:adsk.eagle:package:23617/2"/>
+<part name="C2" library="rcl" library_urn="urn:adsk.eagle:library:334" deviceset="C-EU" device="C0805" package3d_urn="urn:adsk.eagle:package:23617/2"/>
+<part name="GND7" library="supply1" library_urn="urn:adsk.eagle:library:371" deviceset="GND" device=""/>
+<part name="GND8" library="supply1" library_urn="urn:adsk.eagle:library:371" deviceset="GND" device=""/>
 </parts>
 <sheets>
@@
 <attribute name="VALUE" x="-54.61" y="78.74" size="1.778" layer="96" rot="R180"/>
 </instance>
+<instance part="C1" gate="G$1" x="114.3" y="35.56" smashed="yes">
+<attribute name="NAME" x="115.824" y="35.941" size="1.778" layer="95"/>
+<attribute name="VALUE" x="115.824" y="30.861" size="1.778" layer="96"/>
+</instance>
+<instance part="C2" gate="G$1" x="121.92" y="35.56" smashed="yes">
+<attribute name="NAME" x="123.444" y="35.941" size="1.778" layer="95"/>
+<attribute name="VALUE" x="123.444" y="30.861" size="1.778" layer="96"/>
+</instance>
+<instance part="GND7" gate="1" x="114.3" y="15.24" smashed="yes">
+<attribute name="VALUE" x="111.76" y="12.7" size="1.778" layer="96"/>
+</instance>
+<instance part="GND8" gate="1" x="121.92" y="15.24" smashed="yes">
+<attribute name="VALUE" x="119.38" y="12.7" size="1.778" layer="96"/>
+</instance>
 </instances>
 <busses>
@@
 <pinref part="GND6" gate="1" pin="GND"/>
 <wire x1="12.7" y1="93.98" x2="12.7" y2="91.44" width="0.1524" layer="91"/>
+</segment>
+<segment>
+<pinref part="GND7" gate="1" pin="GND"/>
+<pinref part="C1" gate="G$1" pin="2"/>
+<wire x1="114.3" y1="17.78" x2="114.3" y2="30.48" width="0.1524" layer="91"/>
+</segment>
+<segment>
+<pinref part="GND8" gate="1" pin="GND"/>
+<pinref part="C2" gate="G$1" pin="2"/>
+<wire x1="121.92" y1="17.78" x2="121.92" y2="30.48" width="0.1524" layer="91"/>
 </segment>
 </net>
@@
 <pinref part="U$1" gate="G$1" pin="A"/>
 <pinref part="U$2" gate="G$1" pin="PB0"/>
-<wire x1="99.06" y1="33.02" x2="99.06" y2="78.74" width="0.1524" layer="91"/>
+<wire x1="99.06" y1="33.02" x2="99.06" y2="48.26" width="0.1524" layer="91"/>
+<wire x1="99.06" y1="48.26" x2="99.06" y2="78.74" width="0.1524" layer="91"/>
 <wire x1="99.06" y1="78.74" x2="-2.54" y2="78.74" width="0.1524" layer="91"/>
+<pinref part="C2" gate="G$1" pin="1"/>
+<wire x1="121.92" y1="38.1" x2="121.92" y2="48.26" width="0.1524" layer="91"/>
+<wire x1="121.92" y1="48.26" x2="99.06" y2="48.26" width="0.1524" layer="91"/>
+<junction x="99.06" y="48.26"/>
 </segment>
 </net>
@@
 <pinref part="U$1" gate="G$1" pin="B"/>
 <pinref part="U$2" gate="G$1" pin="PB1"/>
-<wire x1="104.14" y1="33.02" x2="104.14" y2="81.28" width="0.1524" layer="91"/>
+<wire x1="104.14" y1="33.02" x2="104.14" y2="43.18" width="0.1524" layer="91"/>
+<wire x1="104.14" y1="43.18" x2="104.14" y2="81.28" width="0.1524" layer="91"/>
 <wire x1="104.14" y1="81.28" x2="-2.54" y2="81.28" width="0.1524" layer="91"/>
+<pinref part="C1" gate="G$1" pin="1"/>
+<wire x1="114.3" y1="38.1" x2="114.3" y2="43.18" width="0.1524" layer="91"/>
+<wire x1="114.3" y1="43.18" x2="104.14" y2="43.18" width="0.1524" layer="91"/>
+<junction x="104.14" y="43.18"/>
 </segment>
 </net>
@@
 packages will not be understood (or retained) with this version.
 </note>
+<note version="8.4" severity="warning">
+Since Version 8.4, EAGLE supports properties for SPICE simulation.
+Probes in schematics and SPICE mapping objects found in parts and library devices
+will not be understood with this version. Update EAGLE to the latest version
+for full support of SPICE simulation.
+</note>
 </compatibility>
