File: v3.0/proudovyzdroj.brd (EAGLE design)
At the start: 160 x 100 mm, 27 parts, among them IC1 LM358N, Q1 IRF512

Commit message: základní schéma
Parts:
- added C6: (no value), rcl:E3,5-8
- added D3: (no value), diode:SMC
- added R11, R12: (no value), rcl:R0805
- added T1: (no value), transistor:TO92-CBE
- added T2: (no value), transistor-neu-to92:TO220V
- added U$5, U$6: MCP4726, DAC:TSOT23-6
- added ZD2: (no value), devices:DO34-5
- D2: value 1N4004 -> (none); device diode:DO41-10 -> diode:SMC
- IC2: value (none) -> LM358N; device v-reg:317TS -> linear:DIL08
- R5: device rcl:PT-10S -> rcl:R0805
- R6: device rcl:PT-10S -> rcl:RTRIM3339P
- moved C2 130.8 mm to (-25.4, -100.3), turned to 0 degrees
- moved R7 129.2 mm to (-27.9, -76.2), flipped to the top, turned to 0 degrees
- moved D2 105.1 mm to (-24.1, -82.5), turned to 0 degrees
- moved IC2 47.9 mm to (-5.08, -40.6), turned to 0 degrees
- moved R8 38.9 mm to (38.1, -6.35), turned to 270 degrees
- moved D1 35.9 mm to (44.5, 34.3)
- moved R6 34.1 mm to (26.7, 6.35), turned to 270 degrees
- moved C3 27.0 mm to (-6.35, 26.7)
- moved R5 22.7 mm to (22.9, 8.89), flipped to the bottom, turned to 180 degrees
- moved ZD1 21.9 mm to (22.9, -12.7), turned to 180 degrees
- moved IC1 16.6 mm to (26.7, 16.5), turned to 180 degrees
- moved C1 14.9 mm to (22.9, 33.0)
- moved R4 13.3 mm to (11.4, 7.62)
- moved R9 2.54 mm to (-6.35, -7.62)
Connections:
- removed net A0: R10.2, R9.1, R9.2
- new net N$13: C1.+, D1.A, R6.3, R9.3, T2.2, X1.2
- new net N$14: R12.1, T2.1
- new net N$15: C3.+, C4.+, C5.+, D1.C, R4.2, T2.3, U$2.P$2, U$4.P$2
- new net N$16: R12.2, R4.1, T1.C
- new net N$4: R11.1, T1.B
- new net SCL: U$5.5, U$6.5
- new net SDA: U$5.4, U$6.4
- net A1: now also IC2.1, R7.2, ZD2.C; no longer IC1.7
- net GND: now also C4.-, C5.-, C6.-, D2.A, D3.A, IC2.4, T1.E, U$1.3, U$1.5, U$3.3, U$3.5, U$5.2, U$6.2, ZD2.A; no longer R6.1
- net N$1: now also IC2.3; no longer IC1.5
- net N$10: now also D3.C
- net N$11: now also IC1.6, R6.1, R6.2; no longer C2.+, D2.A, IC2.1, R4.1, R5.3
- net N$12: now also IC1.7, R11.2; no longer R6.2, R7.1
- net N$3: now also IC2.2; no longer IC1.6
- net N$5: now also R10.2, R7.1, R9.1, R9.2; no longer C1.+, D1.A, D2.C, IC2.2, R4.2, R9.3, X1.2
- net N$6: now also U$5.1; no longer R6.3
- net N$8: now also D2.C
- net N$9: now also IC1.5, U$6.1; no longer C3.+, D1.C, IC2.3, U$2.P$2, U$4.P$2
- net VCC: now also U$5.3, U$5.6, U$6.3, U$6.6; no longer R7.2
- net VCC/2: now also C2.+, C6.+, IC2.8
Routing:
- net VCC/2: track 0.00 -> 44.5 mm
- net N$11: track 39.8 -> 10.0 mm
- net N$2: track 0.00 -> 23.2 mm, vias 0 -> 2
- net N$5: track 18.2 -> 0.00 mm
- net N$13: track 0.00 -> 16.8 mm, vias 0 -> 2
- net N$4: track 0.00 -> 12.3 mm
- net N$9: track 16.6 -> 5.70 mm, vias 0 -> 1
- net GND: track 22.7 -> 12.3 mm
- net N$16: track 0.00 -> 9.74 mm
- net N$12: track 0.00 -> 5.40 mm
- net N$15: track 0.00 -> 4.13 mm
- net N$14: track 0.00 -> 4.13 mm

Commit message: náznak řízení spínané části, úklid schématu
Parts:
- removed ARDUINO_NANO1: (no value), ArduinoNanoV30:ARDUINO_NANO
- added C10, C11, C7, C8, C9: (no value), rcl:C0805
- added Q2, Q3, Q4: BS170, transistor-small-signal:SOT54E
- added R13, R14, R15, R16: (no value), rcl_my:M0805
- C1: value (none) -> 470u
- R1: device rcl:0207/10 -> rcl_my:M0805
- R11: device rcl:R0805 -> rcl_my:M0805
- R2: device rcl:0207/10 -> rcl:RTRIM3339P
- moved R1 219.7 mm to (-36.8, -188.0)
- moved R2 219.7 mm to (-35.6, -177.8)
- moved R11 172.3 mm to (-27.9, -147.3), flipped to the top, turned to 0 degrees
Connections:
- new net N$18: Q3.D, R15.1
- new net N$19: Q4.D, R16.1
- new net N$20: Q2.D, R14.1
- net A1: now also C10.1, R2.3; no longer ARDUINO_NANO1.5, R2.1
- net GND: now also C10.2, C11.2, C7.2, C8.2, C9.2, Q2.S, Q3.S, Q4.S, R13.1; no longer ARDUINO_NANO1.14, ARDUINO_NANO1.19
- net N$12: now also C7.1, T1.B; no longer R11.2
- net N$15: now also R11.2
- net N$2: now also C11.1
- net N$3: now also R2.1
- net N$4: now also R13.2, R14.2, R15.2, R16.2, U$1.4, U$3.4; no longer T1.B
- net VCC: no longer ARDUINO_NANO1.12
- net VCC/2: now also C8.1, C9.1; no longer ARDUINO_NANO1.15
Routing:
- net N$4: track 12.3 -> 0.00 mm
- net N$12: track 5.40 -> 8.15 mm
- net N$13: track 16.8 -> 15.8 mm

Commit message: přidání řízení DAC1 a ADC
Parts:
- removed C2, C4, C5, C6: (no value), rcl:E3,5-8
- removed D2, D3: (no value), diode:SMC
- removed Q2, Q3, Q4: BS170, transistor-small-signal:SOT54E
- removed R11, R13, R14, R15, R16: (no value), rcl_my:M0805
- removed U$1, U$3: AP1501TO220, regulators:TO220-5
- removed U$2, U$4: DTMSSDTMSS-16/0,033/6,0, induktory a trafa:DTMSS-16/0,033/6,0
Connections:
- removed net N$10: D3.C, U$1.2, U$2.P$1
- removed net N$15: C3.+, C4.+, C5.+, D1.C, R11.2, R4.2, T2.3, U$2.P$2, U$4.P$2
- removed net N$18: Q3.D, R15.1
- removed net N$19: Q4.D, R16.1
- removed net N$20: Q2.D, R14.1
- removed net N$4: R11.1, R13.2, R14.2, R15.2, R16.2, U$1.4, U$3.4
- removed net N$8: D2.C, U$3.2, U$4.P$1
- new net N$24: C3.+, D1.C, R4.2, T2.3
- net GND: no longer C2.-, C4.-, C5.-, C6.-, D2.A, D3.A, Q2.S, Q3.S, Q4.S, R13.1, U$1.3, U$1.5, U$3.3, U$3.5
- net VCC/2: no longer C2.+, C6.+, U$1.1, U$3.1
Routing:
- net VCC/2: track 44.5 -> 39.8 mm
- net N$24: track 0.00 -> 4.13 mm
- net N$15: track 4.13 -> 0.00 mm

Commit message: přenesení do fusionu
Parts:
- removed R4, R8: (no value), rcl:R0805
- removed ZD1: (no value), devices:DO34-5
- R5: value (none) -> 1K
- R6: value (none) -> 7K(10K)
Connections:
- removed net N$14: R12.1, T2.1
- removed net N$16: R12.2, R4.1, T1.C
- new net N$4: R12.1, T1.B
- new net N$8: T1.C, T2.1
- net A1: no longer R7.2, ZD2.C
- net A3: now also R7.2, ZD2.C; no longer R8.2, ZD1.C
- net GND: no longer ZD1.A
- net N$12: now also R12.2; no longer T1.B
- net N$13: no longer R9.3
- net N$24: no longer R4.2
- net N$7: now also R9.3; no longer R8.1
Routing:
- net N$16: track 9.74 -> 0.00 mm
- net N$12: track 8.15 -> 3.81 mm
- net N$24: track 4.13 -> 0.00 mm
- net N$14: track 4.13 -> 0.00 mm
Changed lines of the file:
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@@
 <attribute name="VALUE" x="41.656" y="36.322" size="1.27" layer="27" ratio="10" rot="R270"/>
-</element>
-<element name="ZD1" library="devices" package="DO34-5" value="" x="22.86" y="-12.7" smashed="yes" rot="R180">
-<attribute name="NAME" x="24.511" y="-13.97" size="1.27" layer="25" ratio="10" rot="R180"/>
-<attribute name="VALUE" x="24.511" y="-10.16" size="1.27" layer="27" ratio="10" rot="R180"/>
-</element>
-<element name="R8" library="rcl" library_urn="urn:adsk.eagle:library:334" package="R0805" package3d_urn="urn:adsk.eagle:package:23553/2" value="" x="38.1" y="-6.35" smashed="yes" rot="R270">
-<attribute name="NAME" x="39.37" y="-5.715" size="1.27" layer="25" rot="R270"/>
-<attribute name="POPULARITY" value="86" x="38.1" y="-6.35" size="1.778" layer="27" rot="R270" display="off"/>
-<attribute name="SPICEPREFIX" value="R" x="38.1" y="-6.35" size="1.778" layer="27" rot="R270" display="off"/>
-<attribute name="VALUE" x="35.56" y="-5.715" size="1.27" layer="27" rot="R270"/>
 </element>
 <element name="R9" library="rcl" library_urn="urn:adsk.eagle:library:334" package="RTRIM3339P" package3d_urn="urn:adsk.eagle:package:23757/1" value="" x="-6.35" y="-7.62" smashed="yes">
@@
 <attribute name="VALUE" x="-8.636" y="-41.275" size="1.27" layer="27" ratio="10"/>
 </element>
-<element name="R5" library="rcl" library_urn="urn:adsk.eagle:library:334" package="R0805" package3d_urn="urn:adsk.eagle:package:23553/2" value="" x="22.86" y="8.89" smashed="yes" rot="MR180">
+<element name="R5" library="rcl" library_urn="urn:adsk.eagle:library:334" package="R0805" package3d_urn="urn:adsk.eagle:package:23553/2" value="1K" x="22.86" y="8.89" smashed="yes" rot="MR180">
 <attribute name="NAME" x="22.225" y="7.62" size="1.27" layer="26" rot="MR180"/>
 <attribute name="POPULARITY" value="86" x="22.86" y="8.89" size="1.778" layer="28" rot="MR180" display="off"/>
@@
 <attribute name="VALUE" x="22.225" y="11.43" size="1.27" layer="28" rot="MR180"/>
 </element>
-<element name="R6" library="rcl" library_urn="urn:adsk.eagle:library:334" package="RTRIM3339P" package3d_urn="urn:adsk.eagle:package:23757/1" value="" x="26.67" y="6.35" smashed="yes" rot="R270">
+<element name="R6" library="rcl" library_urn="urn:adsk.eagle:library:334" package="RTRIM3339P" package3d_urn="urn:adsk.eagle:package:23757/1" value="7K(10K)" x="26.67" y="6.35" smashed="yes" rot="R270">
 <attribute name="NAME" x="30.875" y="8.865" size="1.27" layer="25" rot="R270"/>
 <attribute name="POPULARITY" value="29" x="26.67" y="6.35" size="1.778" layer="27" rot="R270" display="off"/>
@@
 <attribute name="POPULARITY" value="0" x="15.24" y="12.7" size="1.778" layer="27" display="off"/>
 <attribute name="VALUE" x="12.7" y="9.398" size="1.27" layer="27" ratio="10"/>
-</element>
-<element name="R4" library="rcl" library_urn="urn:adsk.eagle:library:334" package="R0805" package3d_urn="urn:adsk.eagle:package:23553/2" value="" x="11.43" y="7.62" smashed="yes" rot="MR270">
-<attribute name="NAME" x="10.16" y="8.255" size="1.27" layer="26" rot="MR270"/>
-<attribute name="POPULARITY" value="86" x="11.43" y="7.62" size="1.778" layer="28" rot="MR270" display="off"/>
-<attribute name="SPICEPREFIX" value="R" x="11.43" y="7.62" size="1.778" layer="28" rot="MR270" display="off"/>
-<attribute name="VALUE" x="13.97" y="8.255" size="1.27" layer="28" rot="MR270"/>
 </element>
 <element name="T2" library="transistor-neu-to92" library_urn="urn:adsk.eagle:library:397" package="TO220V" package3d_urn="urn:adsk.eagle:package:28746/2" value="" x="13.97" y="0" smashed="yes" rot="R180">
@@
 <signal name="A1">
 <contactref element="IC1" pad="2"/>
-<contactref element="ZD2" pad="C"/>
-<contactref element="R7" pad="2"/>
 <contactref element="IC2" pad="1"/>
 <contactref element="C10" pad="1"/>
 <contactref element="R2" pad="3"/>
 <wire x1="-28.89" y1="-132.08" x2="-33.02" y2="-177.8" width="0" layer="19" extent="1-1"/>
-<wire x1="-26.99" y1="-76.2" x2="-28.89" y2="-132.08" width="0" layer="19" extent="1-1"/>
-<wire x1="-27.94" y1="-71.12" x2="-26.99" y2="-76.2" width="0" layer="19" extent="1-1"/>
-<wire x1="-8.89" y1="-44.45" x2="-27.94" y2="-71.12" width="0" layer="19" extent="1-1"/>
+<wire x1="-8.89" y1="-44.45" x2="-28.89" y2="-132.08" width="0" layer="19" extent="1-1"/>
 <wire x1="27.94" y1="20.32" x2="-8.89" y2="-44.45" width="0" layer="19" extent="1-1"/>
 </signal>
@@
 <contactref element="Q1" pad="D"/>
 <contactref element="X1" pad="1"/>
-<contactref element="R8" pad="1"/>
+<contactref element="R9" pad="3"/>
 <wire x1="35.56" y1="2.54" x2="3.81" y2="45.7454" width="0" layer="19" extent="1-1"/>
-<wire x1="38.1" y1="-5.4" x2="35.56" y2="2.54" width="0" layer="19" extent="1-1"/>
+<wire x1="-3.81" y1="-7.62" x2="35.56" y2="2.54" width="0" layer="19" extent="1-1"/>
 </signal>
 <signal name="GND">
@@
 <contactref element="C3" pad="-"/>
 <wire x1="-6.35" y1="28.448" x2="-10.668" y2="28.448" width="0.1524" layer="16"/>
-<contactref element="ZD1" pad="A"/>
 <contactref element="R10" pad="1"/>
 <contactref element="U$5" pad="2"/>
@@
 <wire x1="-8.89" y1="-26.7" x2="-1.27" y2="-44.45" width="0" layer="19" extent="1-1"/>
 <wire x1="-11.11" y1="-19.05" x2="-8.89" y2="-26.7" width="0" layer="19" extent="1-1"/>
-<wire x1="20.32" y1="-12.7" x2="-11.11" y2="-19.05" width="0" layer="19" extent="1-1"/>
-<wire x1="20.32" y1="7.3" x2="20.32" y2="-12.7" width="0" layer="19" extent="16-16"/>
+<wire x1="20.32" y1="7.3" x2="-11.11" y2="-19.05" width="0" layer="19" extent="1-16"/>
 <wire x1="18.1" y1="12.7" x2="18.1" y2="12.7" width="0" layer="19" extent="1-16"/>
 <wire x1="19.08" y1="17.78" x2="18.1" y2="12.7" width="0" layer="19" extent="1-16"/>
@@
 <wire x1="-7.94" y1="-26.7" x2="-9.84" y2="-24.1" width="0" layer="19" extent="1-1"/>
 </signal>
-<signal name="A3">
-<contactref element="ZD1" pad="C"/>
-<contactref element="R8" pad="2"/>
-<wire x1="25.4" y1="-12.7" x2="38.1" y2="-7.3" width="0" layer="19" extent="1-1"/>
-</signal>
 <signal name="N$11">
 <contactref element="R5" pad="2"/>
@@
 <contactref element="R6" pad="3"/>
 <contactref element="X1" pad="2"/>
-<contactref element="R9" pad="3"/>
 <contactref element="T2" pad="2"/>
 <contactref element="D1" pad="A"/>
@@
 <wire x1="22.86" y1="31.242" x2="44.45" y2="29.21" width="0" layer="19" extent="1-1"/>
 <wire x1="21.59" y1="5.08" x2="22.86" y2="31.242" width="0" layer="19" extent="1-1"/>
-<wire x1="-3.81" y1="-7.62" x2="13.97" y2="2.54" width="0" layer="19" extent="1-1"/>
 <wire x1="3.81" y1="50.7746" x2="22.86" y2="31.242" width="0" layer="19" extent="1-1"/>
-</signal>
-<signal name="N$16">
-<contactref element="T1" pad="C"/>
-<contactref element="R4" pad="1"/>
-<contactref element="R12" pad="2"/>
-<wire x1="16.51" y1="8.57" x2="11.43" y2="8.57" width="0.1524" layer="16"/>
-<wire x1="12.7" y1="12.7" x2="12.7" y2="9.84" width="0.1524" layer="16"/>
-<wire x1="12.7" y1="9.84" x2="11.43" y2="8.57" width="0.1524" layer="16"/>
 </signal>
 <signal name="N$5">
@@
 <contactref element="IC1" pad="7"/>
 <wire x1="27.94" y1="12.7" x2="27.94" y2="16.51" width="0.1524" layer="16"/>
-<contactref element="T1" pad="B"/>
-<wire x1="16.51" y1="16.51" x2="15.24" y2="15.24" width="0.1524" layer="16"/>
-<wire x1="15.24" y1="15.24" x2="15.24" y2="12.7" width="0.1524" layer="16"/>
 <contactref element="C7" pad="1"/>
-<wire x1="15.24" y1="12.7" x2="-28.89" y2="-142.24" width="0" layer="19" extent="1-1"/>
-<wire x1="27.94" y1="16.51" x2="16.51" y2="16.51" width="0" layer="19" extent="16-16"/>
-</signal>
-<signal name="N$14">
-<contactref element="R12" pad="1"/>
-<contactref element="T2" pad="1"/>
-<wire x1="16.51" y1="6.67" x2="16.51" y2="2.54" width="0.1524" layer="16"/>
+<contactref element="R12" pad="2"/>
+<wire x1="16.51" y1="8.57" x2="-28.89" y2="-142.24" width="0" layer="19" extent="1-16"/>
+<wire x1="27.94" y1="12.7" x2="16.51" y2="8.57" width="0" layer="19" extent="16-16"/>
 </signal>
 <signal name="N$24">
-<contactref element="R4" pad="2"/>
 <contactref element="T2" pad="3"/>
 <contactref element="D1" pad="C"/>
 <contactref element="C3" pad="+"/>
-<wire x1="11.43" y1="2.54" x2="11.43" y2="6.67" width="0.1524" layer="16"/>
-<wire x1="11.43" y1="6.67" x2="44.45" y2="39.37" width="0" layer="19" extent="16-16"/>
-<wire x1="-6.35" y1="24.892" x2="11.43" y2="6.67" width="0" layer="19" extent="16-16"/>
+<wire x1="11.43" y1="2.54" x2="44.45" y2="39.37" width="0" layer="19" extent="1-1"/>
+<wire x1="-6.35" y1="24.892" x2="11.43" y2="2.54" width="0" layer="19" extent="1-1"/>
+</signal>
+<signal name="A3">
+<contactref element="ZD2" pad="C"/>
+<contactref element="R7" pad="2"/>
+<wire x1="-27.94" y1="-71.12" x2="-26.99" y2="-76.2" width="0" layer="19" extent="1-1"/>
+</signal>
+<signal name="N$4">
+<contactref element="R12" pad="1"/>
+<contactref element="T1" pad="B"/>
+<wire x1="16.51" y1="6.67" x2="15.24" y2="12.7" width="0" layer="19" extent="16-16"/>
+</signal>
+<signal name="N$8">
+<contactref element="T1" pad="C"/>
+<contactref element="T2" pad="1"/>
+<wire x1="16.51" y1="2.54" x2="12.7" y2="12.7" width="0" layer="19" extent="1-1"/>
 </signal>
 </signals>

Commit message: přidána rozlévaná měď, rozšířena dokumentace
Parts:
- removed C10, C11, C7: (no value), rcl:C0805
- removed C3: (no value), rcl:E3,5-8
- removed T1: (no value), transistor:TO92-CBE
- removed T2: (no value), transistor-neu-to92:TO220V
- added JP1: (no value), pinhead:1X12
- added K1, K2: CB1-P-24V, relay:CB1
- added PAD1, PAD2: (no value), wirepad:3,81/1,4
- added Q2: TIP120, transistor-power:TO220AH
- added R4: 0R1, rcl:0411/15
- Q1: value IRF512 -> TIP120; device transistor-power:TO220BV -> transistor-power:TO220AH
- R3: device rcl:0207/10 -> rcl:R0805
- moved R3 246.9 mm to (-36.8, -193.0)
- moved R7 128.8 mm to (-49.5, -203.2)
- moved Q1 19.2 mm to (16.5, -2.54)
Connections:
- removed net N$24: C3.+, D1.C, T2.3
- new net +24V: K1.87, K2.30
- new net N$10: K1.87A, PAD1.1
- new net N$14: K2.87, PAD2.1
- net A1: no longer C10.1
- net A3: now also R10.2, R9.1, R9.2; no longer R7.2
- net GND: now also R3.1, R4.1; no longer C10.2, C11.2, C3.-, C7.2, R3.2, T1.E
- net N$1: now also Q1.E, R4.2; no longer Q1.S, R3.1
- net N$12: no longer C7.1
- net N$13: now also D1.C, Q2.E, R3.2; no longer D1.A, T2.2
- net N$2: now also R7.2; no longer C11.1, Q1.G
- net N$4: now also Q2.B; no longer T1.B
- net N$5: now also Q1.B; no longer R10.2, R9.1, R9.2
- net N$7: now also D1.A, Q1.C; no longer Q1.D
- net N$8: now also K1.30, Q2.C; no longer T1.C, T2.1
Routing:
- net N$2: track 23.2 -> 0.00 mm, vias 2 -> 0
- net GND: track 12.3 -> 7.64 mm
- net N$13: track 15.8 -> 13.2 mm

Commit message: Přidán obvod řízení výběru zdroje lineárního regulátoru
Parts:
- removed K1, K2: CB1-P-24V, relay:CB1
- added U$1, U$2: V23105-A5305-A201, realatka:V23105-A5305-A201
- added U$3, U$4: NX3008, NEXPERIA :SOT95P240X110-3N
- moved PAD2 356.4 mm to (20.3, 86.4)
- moved PAD1 347.0 mm to (5.08, 86.4)
- moved JP1 273.2 mm to (17.8, 69.8), turned to 180 degrees
Connections:
- removed net VCC: U$5.3, U$5.6, U$6.3, U$6.6
- new net +3V3: JP1.1, U$5.3, U$5.6, U$6.3, U$6.6
- new net N$15: JP1.5
- new net N$16: U$1.16, U$3.3
- new net N$17: U$2.16, U$4.3
- new net N$18: JP1.6
- new net N$19: PAD2.1, U$1.8, U$1.9
- new net PA8: JP1.10, U$4.1
- new net PA9: JP1.9, U$3.1
- new net SCL2: JP1.3, U$6.5
- new net SDA2: JP1.2, U$6.4
- net +24V: now also JP1.12, U$1.1, U$1.13, U$1.4, U$2.1, U$2.11, U$2.6; no longer K1.87, K2.30
- net GND: now also JP1.11, U$3.2, U$4.2
- net N$10: now also U$2.8, U$2.9; no longer K1.87A
- net N$14: now also JP1.4; no longer K2.87, PAD2.1
- net N$8: now also U$2.13, U$2.4; no longer K1.30
- net SCL: now also JP1.8; no longer U$6.5
- net SDA: now also JP1.7; no longer U$6.4
Routing:
- net +24V: track 0.00 -> 84.0 mm
- net PA9: track 0.00 -> 23.1 mm
- net GND: track 7.64 -> 19.8 mm
- net PA8: track 0.00 -> 10.4 mm
- net N$19: track 0.00 -> 8.89 mm
- net N$10: track 0.00 -> 8.89 mm
- net N$8: track 0.00 -> 5.08 mm
- net N$17: track 0.00 -> 2.64 mm
- net N$16: track 0.00 -> 2.64 mm
