File: linearni_zdroj.sch (EAGLE design)
At the start: 36 parts, among them IC1 LM358N, IC2 LM358N, Q1 IRFZ34NAV, Q2 TIP120, Q3 2N7002, Q4 2N7002

Commit message: doku
Other:
- note added: "-"
- moved on the sheet: --2
Changed lines of the file:
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@@
 <wire x1="210.82" y1="266.7" x2="210.82" y2="256.54" width="0.1524" layer="97"/>
 <text x="60.96" y="259.08" size="5.08" layer="97">Deska lineárních regulátorů</text>
+<text x="195.58" y="60.96" size="6.4516" layer="97">-</text>
 </plain>
 <instances>
@@
 <attribute name="NAME" x="191.77" y="62.611" size="1.778" layer="95"/>
 </instance>
-<instance part="-" gate="-2" x="180.34" y="83.82" smashed="yes" rot="R270">
-<attribute name="NAME" x="181.229" y="85.09" size="1.778" layer="95" rot="R90"/>
-<attribute name="VALUE" x="176.657" y="87.63" size="1.778" layer="96" rot="R270"/>
+<instance part="-" gate="-2" x="190.5" y="81.28" smashed="yes" rot="R180">
+<attribute name="NAME" x="191.77" y="80.391" size="1.778" layer="95"/>
+<attribute name="VALUE" x="194.31" y="84.963" size="1.778" layer="96" rot="R180"/>
 </instance>
 <instance part="GND1" gate="1" x="162.56" y="17.78" smashed="yes">
@@
 <pinref part="-" gate="-2" pin="KL"/>
 <pinref part="D1" gate="G$1" pin="C"/>
-<wire x1="180.34" y1="73.66" x2="180.34" y2="78.74" width="0.1524" layer="91"/>
-<label x="175.26" y="76.2" size="3.81" layer="95"/>
+<label x="195.58" y="78.74" size="3.81" layer="95"/>
+<wire x1="180.34" y1="73.66" x2="180.34" y2="81.28" width="0.1524" layer="91"/>
+<wire x1="180.34" y1="81.28" x2="185.42" y2="81.28" width="0.1524" layer="91"/>
 </segment>
 </net>
