File: tlacitka.sch (EAGLE design)
At the start: 7 parts, among them SW1 1825910-6, SW2 1825910-6, SW3 1825910-6

Commit message: doku
Parts:
- SW1, SW2, SW3: value 1825910-6 -> B3F-1000; device Switch:1825910-6 -> Switch:B3F-1000
- renumbered PAD4 to GND
Connections:
- net N$1: now also PAD1.P, SW1.4; no longer GND.P, SW1.1, SW2.2, SW2.4, SW3.2, SW3.4
- net N$2: now also SW2.4; no longer SW2.1
- net N$3: now also GND.P, SW1.1, SW2.1, SW2.2, SW3.1, SW3.2; no longer PAD1.P, SW1.4
- net N$4: now also SW3.4; no longer SW3.1
Other:
- moved on the sheet: SW1, SW2, SW3
